Commit message: Working version (pid parameters might need adjustments)

File: src/mecanum_bot/description/robot.urdf.xacro (robot description, xacro)
@@ -19,5 +19,6 @@
       <visual>
         <geometry>
-          <cylinder radius="0.0485" length="0.03"/> </geometry>
+          <cylinder radius="0.0485" length="0.03"/>
+        </geometry>
         <material name="black"><color rgba="0 0 0 1"/></material>
       </visual>
@@ -30,8 +31,8 @@
     </joint>
   </xacro:macro>
-  <xacro:wheel name="fl" x="0.10"  y="0.12" />
-  <xacro:wheel name="rl" x="-0.10" y="0.12" />
-  <xacro:wheel name="fr" x="0.10"  y="-0.12"/>
-  <xacro:wheel name="rr" x="-0.10" y="-0.12"/>
+  <xacro:wheel name="fl" x="0.0975"  y="0.1035" />
+  <xacro:wheel name="rl" x="-0.0975" y="0.1035" />
+  <xacro:wheel name="fr" x="0.0975"  y="-0.1035"/>
+  <xacro:wheel name="rr" x="-0.0975" y="-0.1035"/>
   <ros2_control name="MecanumTopicBased" type="system">
     <hardware>
@@ -39,4 +40,5 @@
       <param name="port">/dev/ttyACM0</param>
       <param name="baudrate">230400</param>
+      <param name="ticks_per_rev">1980</param>
     </hardware>
     <joint name="fl_wheel_joint">
